File: board/smu2/smu2.kicad_pcb (KiCad board)
At the start: 4 copper layers, 95.2 x 53.3 mm, 201 parts, among them J1 ICD Header, J2 USB4105-GF-A, J3 Left Rails, J4 Right Rails, J5 Analog, J6 Digital, Q1 AOSS21115C, U1 PIC24FJ128GC006-I_MR, U10 AD8420, U11 ADG509F, U12 ADG509F, U13 AD823A, U14 ADG1221, U15 AD8420, U16 AD8420, U17 ADG333A, U18 AD8420, U19 AD8420, U2 ADS8887, U20 ADG509F, U21 ADG509F, U22 AD823A, U23 ADG1221, U24 MCP1702T-3302E_CB, U25 TPS65131-Q1, U26 LT3032EDE-12, U27 MCP6022, U3 ADS8887, U4 DAC8564, U5 RN4871, U6 AD8420, U7 AD8420, U8 ADG333A, U9 AD8420, Y1 32K768

Commit message: Changed R4 from 909Ω to 5.1kΩ
Parts:
- R4: value 909 -> 5.1K
Changed lines of the file:
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@@
 			)
 		)
-		(property "Value" "909"
+		(property "Value" "5.1K"
 			(at 0 1.43 0)
 			(layer "F.Fab")

Commit message: Updated PCB design files.
Parts:
- added C70: 0.1µF, Capacitor_SMD:C_0603_1608Metric, F.Cu at (131.2, 106.7)
- added C71: 0.1µF, Capacitor_SMD:C_0603_1608Metric, F.Cu at (131.2, 124.5)
- added C72: 0.1µF, Capacitor_SMD:C_0603_1608Metric, F.Cu at (128.1, 106.7)
- added C73: 0.1µF, Capacitor_SMD:C_0603_1608Metric, F.Cu at (128.1, 124.5)
- added R75: 1K, Resistor_SMD:R_0603_1608Metric, F.Cu at (131.2, 108.2)
- added R76: 1K, Resistor_SMD:R_0603_1608Metric, F.Cu at (131.2, 126.0)
- added R77: 1K, Resistor_SMD:R_0603_1608Metric, F.Cu at (131.2, 105.2)
- added R78: 1K, Resistor_SMD:R_0603_1608Metric, F.Cu at (131.2, 122.9)
- added R79: 1K, Resistor_SMD:R_0603_1608Metric, F.Cu at (128.1, 108.2)
- added R80: 1K, Resistor_SMD:R_0603_1608Metric, F.Cu at (128.1, 105.2)
- added R81: 1K, Resistor_SMD:R_0603_1608Metric, F.Cu at (128.1, 126.0)
- added R82: 1K, Resistor_SMD:R_0603_1608Metric, F.Cu at (128.1, 122.9)
- moved R38 6.16 mm to (134.2, 124.5), turned to 0 degrees
- moved R42 6.16 mm to (134.2, 126.0), turned to 0 degrees
- moved R13 6.11 mm to (134.2, 106.7), turned to 0 degrees
- moved R17 6.11 mm to (134.2, 108.2), turned to 0 degrees
- moved R44 3.05 mm to (133.2, 110.5), turned to 0 degrees
- moved R50 3.05 mm to (136.3, 113.5), turned to 180 degrees
- moved R45 1.52 mm to (133.2, 112.0)
- moved R46 1.52 mm to (136.3, 110.5)
- moved R47 1.52 mm to (133.2, 113.5), turned to 0 degrees
- moved R49 1.52 mm to (136.3, 112.0)
- moved R14 1.14 mm to (128.1, 103.6)
- moved R26 1.14 mm to (128.1, 102.1)
- moved R39 0.63 mm to (128.1, 121.4)
- moved R51 0.63 mm to (128.1, 119.9)
- moved C19 0.51 mm to (130.4, 100.8)
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Connections:
- R13 pad 1: /CH1IN+ -> Net-(R13-Pad1)
- R15 pad 1: /CH1IN- -> Net-(R15-Pad1)
- R17 pad 1: /CH1IN+ -> Net-(R13-Pad1)
- R18 pad 1: /CH1IN- -> Net-(R15-Pad1)
- R38 pad 1: /CH2IN+ -> Net-(R38-Pad1)
- R40 pad 1: /CH2IN- -> Net-(R40-Pad1)
- R42 pad 1: /CH2IN+ -> Net-(R38-Pad1)
- R43 pad 1: /CH2IN- -> Net-(R40-Pad1)
- U15 pad 8: /CH2IN+ -> Net-(R38-Pad1)
- U16 pad 8: /CH2IN- -> Net-(R40-Pad1)
- U6 pad 8: /CH1IN+ -> Net-(R13-Pad1)
- U7 pad 8: /CH1IN- -> Net-(R15-Pad1)
Routing:
- net Net-(R40-Pad1): track 0.00 -> 12.9 mm, vias 0 -> 2
- net Net-(R15-Pad1): track 0.00 -> 12.3 mm, vias 0 -> 2
- net /CH1IN+: track 16.1 -> 7.64 mm
- net /CH2IN+: track 16.1 -> 8.23 mm
- net Net-(R38-Pad1): track 0.00 -> 6.80 mm
- net Net-(R13-Pad1): track 0.00 -> 6.79 mm
- net /CH2OUT+: track 13.7 -> 8.27 mm
- net /CH1OUT-: track 23.0 -> 28.0 mm
- net /CH1OUT+: track 21.4 -> 25.9 mm
- net Net-(C70-Pad2): track 0.00 -> 3.69 mm
- net Net-(C71-Pad2): track 0.00 -> 3.67 mm
- net /CH1IN-: track 11.1 -> 7.77 mm
- net Net-(R38-Pad2): track 9.17 -> 12.3 mm
- net Net-(R13-Pad2): track 8.91 -> 12.0 mm
- net /CH2IN-: track 11.0 -> 8.01 mm
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Other:
- board text added: "6/21/2025"
- board text removed: "5/29/2025"
