File: board/smu2/smu2.kicad_sch (KiCad schematic)
At the start: 59 parts, among them J1 ICD Header, J2 USB4105-GF-A, J3 Left Rails, J4 Right Rails, J5 Analog, J6 Digital, U1 PIC24FJ128GC006-I_MR, U2 ADS8887, U27 MCP6022, U3 ADS8887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

Commit message: Changed R4 from 909Ω to 5.1kΩ
Parts:
- R4: value 909 -> 5.1K
Changed lines of the file:
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@@
 			)
 		)
-		(property "Value" "909"
+		(property "Value" "5.1K"
 			(at 53.34 146.0499 0)
 			(effects
