File: board/smu2/smu_channel.kicad_sch (KiCad schematic)
At the start: 53 parts, among them U15 AD8420, U16 AD8420, U17 ADG333A, U18 AD8420, U19 AD8420, U20 ADG509F, U21 ADG509F, U22 AD823A, U23 ADG1221

Commit message: Updated PCB design files.
Parts:
- added C70, C72: 0.1µF, Capacitor_SMD:C_0603_1608Metric, symbol Device:C
- added R75, R77, R79, R80: 1K, Resistor_SMD:R_0603_1608Metric, symbol Device:R
Connections:
- net IN+: now also C72.1, R79.1; no longer R38.1, R42.1, U15.8
- net IN-: now also C72.2, R80.1; no longer R40.1, R43.1, U16.8
- new net: R38.1, R42.1, R75.2, U15.8
- new net: R40.1, R43.1, R77.2, U16.8
- new net: C70.2, R77.1, R80.2
- new net: C70.1, R75.1, R79.2
Other:
- moved on the sheet: C37, C38, C39, C40, C41, C42, C43, C44, C45, C46, C47, C48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
